File: SHEMP Cape/NILMCape.brd (EAGLE design)
At the start: 100 x 100 mm, 88 parts, among them U1 ADS8568_PM_64, U10 SI8663BC-B-IS1, U11 SI8663BC-B-IS1, U12 SI8663BC-B-IS1, U13 SI8663BC-B-IS1, U14 SN74CBT16390_DGG, U2 ACS756KCA-050B-PFF-T, U3 SI8663BC-B-IS1, U4 SN74CBT16390_DGG, U5 TPS84250_RKG_41, U6 TPS7A3301_RGW_20, U7 LP2950-33_KVU_3, U8 SI8663BC-B-IS1, U9 TL074_PW_14

Commit message: More schematic capture work.
Parts:
- moved C37 215.7 mm to (-96.5, 14.0)
- moved C41 214.8 mm to (-96.5, -1.27)
- moved C36 214.1 mm to (-96.5, 29.2)
- moved C35 213.2 mm to (-96.5, 41.9)
- moved C43 212.1 mm to (-96.5, 26.7)
- moved C10 211.3 mm to (-121.9, 67.3)
- moved C11 211.3 mm to (-121.9, 97.8)
- moved C5 211.3 mm to (-121.9, 87.6)
- moved C6 211.3 mm to (-118.1, 87.6)
- moved C7 211.3 mm to (-121.9, 82.5)
- moved C9 211.3 mm to (-118.1, 82.5)
- moved R1 211.3 mm to (-121.9, 77.5)
- moved R10 211.3 mm to (-121.9, 92.7)
- moved R13 211.3 mm to (-121.9, 62.2)
- moved R14 211.3 mm to (-121.9, 57.1)
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Connections:
- removed net N$100: U$1.77
- removed net N$86: U$1.58
- removed net N$87: U$1.73
- removed net N$88: U$1.71
- removed net N$89: U$1.69
- removed net N$93: U$1.61
- removed net N$94: U$1.88
- removed net N$95: U$1.67
- removed net N$96: U$1.68
- removed net N$97: U$1.57
- removed net N$98: U$1.59
- removed net N$99: U$1.75
- net BB_DB0: now also U$1.57
- net BB_DB1: now also U$1.59
- net BB_DB10: now also U$1.60
- net BB_DB11: now also U$1.62
- net BB_DB12: now also U$1.68
- net BB_DB13: now also U$1.70
- net BB_DB14: now also U$1.72
- net BB_DB15: now also U$1.88
- net BB_DB2: now also U$1.61
- net BB_DB3: now also U$1.67
- net BB_DB4: now also U$1.69
- net BB_DB5: now also U$1.71
- net BB_DB6: now also U$1.73
- net BB_DB7: now also U$1.75
- net BB_DB8: now also U$1.77
- net BB_DB9: now also U$1.58

Commit message: More Schematic Capture
Parts:
- removed LED1, LED2: (no value), SensorCape:LED-0805
- added C46, C47, C48, C53, C54, C56: 10uF, SensorCape:1210
- added C49, C50, C72, C73, C74: 10nF, SensorCape:0805
- added C51, C52: 10uF, SensorCape:1206
- added C55, C57, C59, C60, C61, C62, C63, C64, C65, C66, C67, C68, C69, C70, C71, C75: .1uF, SensorCape:0805
- added C58: 1uF, SensorCape:0805
- added R25: 499k, ASL:0805
- added R26: 154k, ASL:0805
- added R27: 0, SensorCape:0805
- added U$4, U$5, U$6, U$7: MAX548X, SensorCape:TSSOP14_MC
- added U15: TPS7A4901_DGN_8, SensorCape:DGN8_1P89X1P57
- added U16: SI8660BC-B-IS1, SensorCape:SOIC-16
- R14: value 1k -> 0
- moved R14 227.5 mm to (-130.8, -170.2)
Connections:
- removed net AGND: C3.1, C4.1, C7.1, C9.1, R2.2, R5.2, R8.2, R9.2, U9.12, U9.5
- removed net N$17: R13.2, R14.2, U9.13
- removed net N$22: U1.45
- removed net N$23: U1.48
- removed net N$24: U1.51
- removed net N$25: U1.52
- removed net N$27: U1.58
- removed net N$28: U1.61
- removed net N$29: U1.62
- removed net N$8: U1.4
- removed net SIGNAL_TO_AA: R14.1, U9.14
- new net AA1_R_IN: R27.1, U$4.10
- new net AA1_R_OUT: C73.2, U$4.11, U1.42
- new net AA2_R_IN: U$5.10
- new net AA2_R_OUT: C74.2, U$5.11, U1.47
- new net AA3_R_IN: U$7.10, U2.3
- new net AA3_R_OUT: C72.2, U$7.11, U1.49
- new net BBGND: C70.2, U$1.1, U$1.2, U$1.47, U$1.48, U$1.89, U$1.90, U$1.91, U$1.92, U16.8
- new net BBVDD3V3: C70.1, U$1.49, U16.1
- new net BUSY: U1.35
- new net CONV_A: U1.37
- new net CONV_B: U1.38
- new net CONV_C: U1.39
- new net CONV_D: U1.40
- new net CS*: U1.13
- new net GAIN_R_IN: R13.2, R14.1, U$6.10, U9.13
- new net GAIN_R_OUT: R14.2, R27.2, U$6.11, U9.14
- new net HOT_TO_LOAD: U2.A1, U2.A2, U2.A3, U2.A4, U2.A5
- new net N$86: C49.1, U15.6
- new net N$87: C46.2, U1.6
- new net N$89: C50.2, R25.1, R26.2, U15.2
- new net N$93: C53.2, U1.43
- new net N$94: C48.2, U1.50
- new net N$96: C47.1, U1.63
- new net RD*: U1.12
- new net VDD5V0_A: C50.1, C51.1, C59.1, C60.1, C61.2, C62.2, C64.1, C71.1, C75.1, R25.2, U1.14, U1.4, U1.45, U1.52, U1.57, U1.61, U15.1, U2.2
- new net WR*: U1.11
- net GND: now also C3.1, C4.1, C46.1, C47.2, C48.1, C49.2, C51.2, C52.2, C53.1, C54.1, C55.1, C56.1, C57.1, C58.2, C59.2, C60.2, C61.1, C62.1, C63.2, C64.2, C65.1, C66.1, C67.1, C68.1, C69.1, C7.1, C71.2, C72.1, C73.1, C74.1, C75.2, C9.1, R2.2, R26.1, R5.2, R8.2, R9.2, U$4.14, U$4.2, U$5.14, U$5.2, U$6.14, U$6.2, U$7.14, U$7.2, U1.10, U1.15, U1.2, U1.25, U1.3, U1.34, U1.36, U1.44, U1.46, U1.5, U1.51, U1.53, U1.54, U1.55, U1.58, U1.59, U1.60, U1.62, U1.64, U1.7, U1.8, U15.4, U15.EPAD, U16.9, U2.1, U9.12, U9.5; no longer U$1.1, U$1.2, U$1.47, U$1.48, U$1.89, U$1.90, U$1.91, U$1.92
- net HOT_IN: now also U2.B1, U2.B2, U2.B3, U2.B4, U2.B5
- net HVDD_12A: now also C54.2, C55.2, U1.1
- net HVDD_15D: now also C52.1, U15.5, U15.8
- net HVSS: no longer U1.1
- net HVSS_12A: now also C56.2, C57.2, U1.48
- net N$12: now also U$6.3, U16.11; no longer U1.5
- net N$19: now also U$5.3, U16.12; no longer U1.15
- net N$20: now also U$7.3, U16.10; no longer U1.24
- net N$21: now also U$4.4, U$5.4, U$6.4, U$7.4, U16.14; no longer U1.44
- net N$26: now also U$4.5, U$5.5, U$6.5, U$7.5, U16.13; no longer U1.57
- net N$6: now also U$4.3, U16.15; no longer U1.25
- net N$7: now also C63.1, U1.56; no longer U1.14
- net VDD3V3_D: now also C58.1, C65.2, C66.2, C67.2, C68.2, C69.2, U$4.1, U$4.6, U$5.1, U$5.6, U$6.1, U$6.6, U$7.1, U$7.6, U1.24, U1.41, U1.9, U16.16
- net VDD_3V3EXP: no longer U$1.49
