File: SHEMP Cape/NILMCape.sch (EAGLE design)
At the start: 88 parts, among them U1 ADS8568_PM_64, U10 SI8663BC-B-IS1, U11 SI8663BC-B-IS1, U12 SI8663BC-B-IS1, U13 SI8663BC-B-IS1, U14 SN74CBT16390_DGG, U2 ACS756KCA-050B-PFF-T, U3 SI8663BC-B-IS1, U4 SN74CBT16390_DGG, U5 TPS84250_RKG_41, U6 TPS7A3301_RGW_20, U7 LP2950-33_KVU_3, U8 SI8663BC-B-IS1, U9 TL074_PW_14

Commit message: More Schematic Capture
Parts:
- removed LED1, LED2: (no value), SensorCape:LED0805
- added C46, C47, C48, C53, C54, C56: 10uF, SensorCape:CAP1210
- added C49, C50, C72, C73, C74: 10nF, SensorCape:CAP0805
- added C51, C52: 10uF, SensorCape:CAP1206
- added C55, C57, C59, C60, C61, C62, C63, C64, C65, C66, C67, C68, C69, C70, C71, C75: .1uF, SensorCape:CAP0805
- added C58: 1uF, SensorCape:CAP0805
- added R25: 499k, ASL:RESISTOR0805-RES
- added R26: 154k, ASL:RESISTOR0805-RES
- added R27: 0, SensorCape:RESISTOR0805-RES
- added U$4, U$5, U$6, U$7: MAX548X, SensorCape:MAX548X
- added U15: TPS7A4901_DGN_8, SensorCape:TPS7A4901_DGN_8
- added U16: SI8660BC-B-IS1, SensorCape:SI8660BC-B-IS1
- R14: value 1k -> 0
Connections:
- removed net AGND: C3.1, C4.1, C7.1, C9.1, R2.2, R5.2, R8.2, R9.2, U9.2IN+, U9.4IN+
- removed net N$17: R13.2, R14.2, U9.4IN-
- removed net N$22: U1.AVDD_4
- removed net N$23: U1.HVDD
- removed net N$24: U1.AGND_5
- removed net N$25: U1.AVDD_5
- removed net N$27: U1.AGND_6
- removed net N$28: U1.AVDD
- removed net N$29: U1.AGND
- removed net N$8: U1.AVDD_2
- removed net SIGNAL_TO_AA: R14.1, U9.4OUT
- new net AA1_R_IN: R27.1, U$4.L
- new net AA1_R_OUT: C73.2, U$4.W, U1.CH_A0
- new net AA2_R_IN: U$5.L
- new net AA2_R_OUT: C74.2, U$5.W, U1.CH_A1
- new net AA3_R_IN: U$7.L, U2A.VIOUT
- new net AA3_R_OUT: C72.2, U$7.W, U1.CH_B0
- new net BBGND: C70.2, U$1.GND@1, U$1.GND@2, U$1.GND@3, U$1.GND@4, U$1.GND@5, U$1.GND@6, U$1.GND@7, U$1.GND@8, U16.GND1
- new net BBVDD3V3: C70.1, U$1.VDD_3V3EXP@1, U16.VDD1
- new net BUSY: U1.BUSY/INT
- new net CONV_A: U1.CONVST_A
- new net CONV_B: U1.CONVST_B
- new net CONV_C: U1.CONVST_C
- new net CONV_D: U1.CONVST_D
- new net CS*: U1.*CS/*FS
- new net GAIN_R_IN: R13.2, R14.1, U$6.L, U9.4IN-
- new net GAIN_R_OUT: R14.2, R27.2, U$6.W, U9.4OUT
- new net HOT_TO_LOAD: U2B.IP+
- new net N$86: C49.1, U15.NR/SS
- new net N$87: C46.2, U1.REFDP
- new net N$89: C50.2, R25.1, R26.2, U15.FB
- new net N$93: C53.2, U1.REFAP
- new net N$94: C48.2, U1.REFBP
- new net N$96: C47.1, U1.REFCP
- new net RD*: U1.*RD
- new net VDD5V0_A: C50.1, C51.1, C59.1, C60.1, C61.2, C62.2, C64.1, C71.1, C75.1, R25.2, U1.AVDD, U1.AVDD_2, U1.AVDD_3, U1.AVDD_4, U1.AVDD_5, U1.AVDD_6, U15.OUT, U2A.VCC
- new net WR*: U1.REFEN/*WR
- net GND: now also C3.1, C4.1, C46.1, C47.2, C48.1, C49.2, C51.2, C52.2, C53.1, C54.1, C55.1, C56.1, C57.1, C58.2, C59.2, C60.2, C61.1, C62.1, C63.2, C64.2, C65.1, C66.1, C67.1, C68.1, C69.1, C7.1, C71.2, C72.1, C73.1, C74.1, C75.2, C9.1, R2.2, R26.1, R5.2, R8.2, R9.2, U$4.GND, U$4.VSS, U$5.GND, U$5.VSS, U$6.GND, U$6.VSS, U$7.GND, U$7.VSS, U1.*PAR/SER, U1.AGND, U1.AGND_2, U1.AGND_3, U1.AGND_4, U1.AGND_5, U1.AGND_6, U1.ASLEEP, U1.CH_B1, U1.CH_C0, U1.CH_C1, U1.CH_D0, U1.CH_D1, U1.DVDD, U1.RANGE/XCLK, U1.REFAN, U1.REFBN, U1.REFCN, U1.REFDN, U1.REFN, U1.RESET, U15.EPAD, U15.GND, U16.GND2, U2A.GND, U9.2IN+, U9.4IN+
- net HOT_IN: now also U2B.IP-
- net HVDD_12A: now also C54.2, C55.2, U1.HVSS
- net HVDD_15D: now also C52.1, U15.EN, U15.IN
- net HVSS: no longer U1.HVSS
- net HVSS_12A: now also C56.2, C57.2, U1.HVDD
- net N$12: now also U$6.CS*, U16.B5; no longer U1.AGND_2
- net N$19: now also U$5.CS*, U16.B4; no longer U1.AGND_3
- net N$20: now also U$7.CS*, U16.B6; no longer U1.DGND
- net N$21: now also U$4.SCLK, U$5.SCLK, U$6.SCLK, U$7.SCLK, U16.B2; no longer U1.AGND_4
- net N$26: now also U$4.DIN, U$5.DIN, U$6.DIN, U$7.DIN, U16.B3; no longer U1.AVDD_6
- net N$6: now also U$4.CS*, U16.B1; no longer U1.DVDD
- net N$7: now also C63.1, U1.REFIO; no longer U1.AVDD_3
- net VDD3V3_D: now also C58.1, C65.2, C66.2, C67.2, C68.2, C69.2, U$4.SPI/UD*, U$4.VDD, U$5.SPI/UD*, U$5.VDD, U$6.SPI/UD*, U$6.VDD, U$7.SPI/UD*, U$7.VDD, U1.*HW/SW, U1.*STBY, U1.DGND, U16.VDD2
Other:
- note added: "10k Digital Pot"
- note added: "50k Digital Pot"
- note added: "60Hz Filter/Current Sensor"
- note added: "ADC Mux"
- note added: "BeagleBone Mux"
- note added: "DIGITAL POTENTIOMETERS"
- note added: "Data Bus Digital Isolation"
- note removed: "60Hz Filter"
- note removed: "Digital Isolation"
- note removed: "Digital Pot Goes Here"
