File: SEAD Hardware/ADC Module/Eagle Files/ADCModule.sch (EAGLE design)
At the start: 49 parts, among them IC2 93-C46AST, U1 LP2989_DGK_8, X1 52885-0374

Commit message: More layout work.
Connections:
- removed net N$24: C18.2, C7.1, U1.GND
- net GND: now also C18.2, C7.1, U1.GND
Changed lines of the file:
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@@
-</segment>
-<segment>
-<pinref part="USB1" gate="USB" pin="GND"/>
-<wire x1="58.42" y1="195.58" x2="63.5" y2="195.58" width="0.1524" layer="91"/>
-<wire x1="63.5" y1="195.58" x2="63.5" y2="200.66" width="0.1524" layer="91"/>
-<label x="63.5" y="208.28" size="1.778" layer="95"/>
-<pinref part="C6" gate="G$1" pin="1"/>
-<wire x1="63.5" y1="200.66" x2="63.5" y2="208.28" width="0.1524" layer="91"/>
-<junction x="63.5" y="200.66"/>
 </segment>
 <segment>
@@
 <label x="132.08" y="210.82" size="1.778" layer="95"/>
 </segment>
+<segment>
+<pinref part="U1" gate="A" pin="GND"/>
+<pinref part="C7" gate="G$1" pin="1"/>
+<pinref part="C18" gate="G$1" pin="2"/>
+<wire x1="96.52" y1="45.72" x2="96.52" y2="48.26" width="0.1524" layer="91"/>
+<wire x1="96.52" y1="48.26" x2="96.52" y2="53.34" width="0.1524" layer="91"/>
+<wire x1="106.68" y1="48.26" x2="96.52" y2="48.26" width="0.1524" layer="91"/>
+<junction x="96.52" y="48.26"/>
+</segment>
+<segment>
+<pinref part="C6" gate="G$1" pin="1"/>
+<wire x1="63.5" y1="200.66" x2="63.5" y2="208.28" width="0.1524" layer="91"/>
+<junction x="63.5" y="200.66"/>
+<wire x1="63.5" y1="195.58" x2="63.5" y2="200.66" width="0.1524" layer="91"/>
+<pinref part="USB1" gate="USB" pin="GND"/>
+<wire x1="58.42" y1="195.58" x2="63.5" y2="195.58" width="0.1524" layer="91"/>
+<label x="63.5" y="208.28" size="1.778" layer="95"/>
+</segment>
 </net>
 <net name="N$8" class="0">
@@
 </segment>
 </net>
-<net name="N$24" class="0">
-<segment>
-<pinref part="U1" gate="A" pin="GND"/>
-<pinref part="C7" gate="G$1" pin="1"/>
-<pinref part="C18" gate="G$1" pin="2"/>
-<wire x1="96.52" y1="45.72" x2="96.52" y2="48.26" width="0.1524" layer="91"/>
-<wire x1="96.52" y1="48.26" x2="96.52" y2="53.34" width="0.1524" layer="91"/>
-<wire x1="106.68" y1="48.26" x2="96.52" y2="48.26" width="0.1524" layer="91"/>
-<junction x="96.52" y="48.26"/>
-</segment>
-</net>

Commit message: Finished DAQ revision.
Parts:
- added C25, C26, C27, C28: .1uF, SensorCape:CAP0805
Connections:
- net VDD1V8_D renamed VCC1V8_D
- net CANRX: no longer X1-7.S
- net CANTX: no longer X1-9.S
- net GND: now also C25.1, C26.1, C27.1, C28.1
- net VDD3V3_D: now also C25.2, C26.2, C27.2, C28.2
