File: SEAD Hardware/ADC Module/Eagle Files/ADCModule.sch (EAGLE design)
At the start: 53 parts, among them IC2 93-C46AST, U1 LP2989_DGK_8, X1 52885-0374

Commit message: Started ADC Hat. Library additions.
Changed lines of the file:
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@@
-</segment>
-<segment>
-<wire x1="264.16" y1="218.44" x2="261.62" y2="218.44" width="0.1524" layer="91"/>
-<label x="259.08" y="218.44" size="1.778" layer="95"/>
 </segment>
 <segment>
@@
 </segment>
 <segment>
-<wire x1="264.16" y1="236.22" x2="259.08" y2="236.22" width="0.1524" layer="91"/>
-<label x="264.16" y="236.22" size="1.778" layer="95" rot="MR0"/>
-</segment>
-<segment>
 <pinref part="X1" gate="-10" pin="S"/>
 <wire x1="231.14" y1="243.84" x2="228.6" y2="243.84" width="0.1524" layer="91"/>
@@
 </segment>
 <segment>
-<wire x1="264.16" y1="241.3" x2="259.08" y2="241.3" width="0.1524" layer="91"/>
-<label x="259.08" y="241.3" size="1.778" layer="95"/>
-</segment>
-<segment>
 <pinref part="X1" gate="-6" pin="S"/>
 <wire x1="231.14" y1="248.92" x2="228.6" y2="248.92" width="0.1524" layer="91"/>
@@
 </segment>
 <segment>
-<wire x1="264.16" y1="243.84" x2="259.08" y2="243.84" width="0.1524" layer="91"/>
-<label x="259.08" y="243.84" size="1.778" layer="95"/>
-</segment>
-<segment>
 <pinref part="X1" gate="-4" pin="S"/>
 <wire x1="231.14" y1="251.46" x2="228.6" y2="251.46" width="0.1524" layer="91"/>
@@
 <wire x1="40.64" y1="119.38" x2="45.72" y2="119.38" width="0.1524" layer="91"/>
 <label x="48.26" y="119.38" size="1.778" layer="95"/>
-</segment>
-<segment>
-<wire x1="264.16" y1="238.76" x2="259.08" y2="238.76" width="0.1524" layer="91"/>
-<label x="259.08" y="238.76" size="1.778" layer="95"/>
 </segment>
 <segment>
@@
 </segment>
 </net>
-<net name="N$3" class="0">
-<segment>
-<wire x1="259.08" y1="246.38" x2="264.16" y2="246.38" width="0.1524" layer="91"/>
-</segment>
-</net>
-<net name="N$6" class="0">
-<segment>
-<wire x1="259.08" y1="248.92" x2="264.16" y2="248.92" width="0.1524" layer="91"/>
-</segment>
-</net>
-<net name="N$7" class="0">
-<segment>
-<wire x1="259.08" y1="251.46" x2="264.16" y2="251.46" width="0.1524" layer="91"/>
-</segment>
-</net>
