File: SEAD Hardware/ADC Module/Eagle Files/Hat_MCP3912.sch (EAGLE design)
At the start: 36 parts, among them IC1 MCP3912, X2 52885-0374

Commit message: More board work.
Parts:
- removed X2: 52885-0374, SensorCape:52885-0374
- added C10: .01uF, SensorCape:CAP0805
- added C11, C12: 20pF, SensorCape:CAP0805
- added C18: 2.2uF, SensorCape:CAP0805
- added C19: 4.7uF, SensorCape:CAP0805
- added U$1: 7M-12.000MEEQ-T, SensorCape:7M-12.000MEEQ-T
- added U1: LP2989_DGK_8, SensorCape:LP2989_DGK_8
- added X1: 55091-0374, SensorCape:55091-0374
Connections:
- new net N$24: C10.2, U1.BYPASS
- new net N$26: C11.1, IC1.OSC2, U$1.OSC2
- new net N$27: C12.2, IC1.OSC1/CLKI, U$1.OSC1
- net AGND: now also C19.1, JP1.2, JP2.2, JP3.2, JP4.2
- net GND: now also C10.1, C11.2, C12.1, C18.2, U$1.GND1, U$1.GND2, U1.GND, X1-1.S, X1-12.S, X1-18.S, X1-2.S, X1-24.S, X1-29.S, X1-30.S; no longer X2-1.S, X2-11.S, X2-17.S, X2-2.S, X2-23.S, X2-29.S, X2-30.S
- net MISO: now also X1-4.S; no longer X2-3.S
- net MOSI: now also X1-6.S; no longer X2-5.S
- net SCK: now also X1-10.S; no longer X2-9.S
- net SCL: now also X1-16.S; no longer X2-15.S
- net SDA: now also X1-14.S; no longer X2-13.S
- net SS: now also X1-8.S; no longer X2-7.S
- net U1RX: now also X1-22.S; no longer X2-21.S
- net U1TX: now also X1-20.S; no longer X2-19.S
- net U3RX: now also X1-28.S; no longer X2-27.S
- net U3TX: now also X1-26.S; no longer X2-25.S
- net VDD3V3_A: now also C19.2, U1.SENSE, U1.VOUT
- net VDD3V3_D: now also X1-5.S; no longer X2-6.S
- net VDD5V0_D: now also C18.1, U1.VIN, U1.~SD, X1-3.S; no longer X2-4.S
Other:
- note removed: "Put down a 16MHz Crystal!!!"
