File: SEAD Hardware/Power Supply/Split12VoltForTesting.sch (EAGLE design)
At the start: 2 parts, among them U1 LM2575_N_16

Commit message: Finished quick power supply.
Parts:
- removed U1: LM2575_N_16, SensorCape:LM2575_N_16
- added C1, C4, C5, C7: 2.2uF, SensorCape:CAP1210
- added C2, C3, C6: 100uF, SensorCape:CAP_POLPTH1
- added JP1, JP2: M03LONGPADS, SensorCape:M03LONGPADS
- added LED1, LED2: (no value), SensorCape:LED0805
- added R1: 14.9k, SensorCape:RESISTOR0805-RES
- added R2: 100, SensorCape:RESISTOR0805-RES
- added R3, R4: 1.5k, SensorCape:RESISTOR0805-RES
- added U$2: PTN78060A, SensorCape:PTN78060A
- U$1: device ASL:PTN78000THROUGH-HOLE -> SensorCape:PTN78000THROUGH-HOLE
Connections:
- removed net VCC12V0_D: U1.VIN
- new net N$1: LED2.C, R3.1
- new net N$2: R2.2, U$2.VOADJUST
- new net N$3: R1.2, U$1.ADJ
- new net N$4: LED1.C, R4.2
- new net VDD15V0_D: C2.+, C3.+, C4.1, C5.1, JP1.3, LED1.A, U$1.V_OUT, U$2.VIN
- new net VSS15V0_D: C5.2, C6.-, C7.2, JP1.1, LED2.A, R2.1, U$2.V_OUT1, U$2.V_OUT2
- new net V_IN: C1.1, JP2.1, U$1.V_IN
- net GND: now also C1.2, C2.-, C3.-, C4.2, C6.+, C7.1, JP1.2, JP2.2, JP2.3, R1.1, R3.2, R4.1, U$1.GND, U$2.GND; no longer U1.GND_2, U1.GND_3
Other:
- note added: "Slightly Larger Is Better"
- moved on the sheet: U$1
