File: Hardware/PIC32 Based Hardware/SEAD Light/AFE_Pants_Powered.sch (EAGLE design)
At the start: 43 parts, among them IC1 MCP3912, U1 LP2989_DGK_8, X1 55091-0374

Commit message: Added gerbers and layouts.
Parts:
- removed JP1, JP2, JP3, JP4: M03LONGPADS, SensorCape:M03LONGPADS
- added C13: 10nF, SensorCape:CAP0805
- added R22, R23: 332000, SensorCape:RESISTOR0805-RES
- added R24: 1000, SensorCape:RESISTOR0805-RES
- added U$2: ECE05US05, SensorCape:ECE05US05
- added X2: (no value), con-wago-500:W237-6
- added X3: (no value), con-wago-500:W237-103
Connections:
- removed net N$22: IC1.CH3-, JP4.1
- new net N$28: R23.1, U$2.ACL, X3-1.KL
- new net N$29: U$2.ACN, X3-3.KL
- new net N$30: R22.1, R23.2
- net AGND: no longer JP1.2, JP2.2, JP3.2, JP4.2
- net GND: now also C13.1, IC1.CH3-, R24.2, U$2.-V
- net N$10: now also X2-2.KL; no longer JP1.1
- net N$11: now also X2-1.KL; no longer JP1.3
- net N$12: now also X2-4.KL; no longer JP2.1
- net N$15: now also X2-3.KL; no longer JP2.3
- net N$18: now also X2-6.KL; no longer JP3.1
- net N$19: now also X2-5.KL; no longer JP3.3
- net N$23: now also C13.2, R22.2, R24.1; no longer JP4.3
- net VDD5V0_D: now also U$2.+V
