File: Hardware/PIC32 Based Hardware/SEAD Light/SEADLight.brd (EAGLE design)
At the start: 45 x 36.5 mm, 53 parts, among them IC2 93-C46AST, U1 LP2989_DGK_8, X1 52885-0374

Commit message: Added gerbers and layouts.
Parts:
- removed C20: 3.3uF, SensorCape:EIA3216
- removed C21, C22: 4.7uF, SensorCape:EIA3216
- removed C23, C24, C25, C26, C27, C28, C5: .1uF, SensorCape:0805
- removed C4: 20pF, SensorCape:0805
- removed C6: 100uF, SensorCape:1206
- removed IC1: (no value), SensorCape:LQFP64
- removed IC2: 93-C46AST, microchip:TSSOP8
- removed L1, L2: (no value), dp_devices.v6:FB805
- removed LED2, LED3: (no value), led:CHIP-LED0805
- removed R10, R11: 470, SensorCape:0805
- removed R4, R5, R6, R8: 10k, SensorCape:0805
- removed R7: 2.2k, SensorCape:0805
- removed R9: 12k 1%, SensorCape:0805
- removed USB1: CON-USB-F-MICRO-B, dp_devices.v6:CONN_USB_MICRO-B
- C3: value 20pF -> 4.7uF
- U$3: value 7M-12.000MEEQ-T -> EPS8266; device SensorCape:7M-CRYSTAL -> SensorCape:ESP8266-03
- moved C3 24.5 mm to (19.5, 30.0), turned to 90 degrees
- moved C19 9.72 mm to (12.2, 10.2), turned to 270 degrees
- moved C7 8.56 mm to (4.34, 10.2), turned to 90 degrees
- moved U1 7.11 mm to (8.24, 10.1), turned to 0 degrees
- moved C18 5.01 mm to (5.44, 7.87), turned to 180 degrees
- moved U$3 3.45 mm to (4.50, 18.0), turned to 0 degrees
Connections:
- removed net A0: IC1.27, U$1.44
- removed net CANRX: U$1.87
- removed net CANTX: U$1.88
- removed net CS*: IC1.26, U$1.71
- removed net D0: IC1.16, U$1.93
- removed net D1: IC1.17, U$1.94
- removed net D2: IC1.18, U$1.98
- removed net D3: IC1.19, U$1.99
- removed net D4: IC1.21, U$1.100
- removed net D5: IC1.22, U$1.3
- removed net D6: IC1.23, U$1.4
- removed net D7: IC1.24, U$1.5
- removed net N$10: IC1.7, USB1.P2
- removed net N$11: IC1.8, USB1.P3
- removed net N$12: IC1.63, IC2.1, R4.1
- removed net N$13: IC1.62, IC2.2, R5.1
- removed net N$17: IC2.4, R6.1, R7.1
- removed net N$18: IC1.61, IC2.3, R7.2
- removed net N$19: IC1.14, R8.1
- removed net N$20: IC1.6, R9.1
- removed net N$21: C22.A, C24.1, IC1.4, L2.1
- removed net N$22: C21.A, C23.1, IC1.9, L1.1
- removed net N$27: IC1.48
- removed net N$28: IC1.54, R10.2
- removed net N$29: IC1.55, R11.2
- removed net N$32: LED2.C, R10.1
- removed net N$33: LED3.C, R11.1
- removed net N$8: C3.1, IC1.3, U$3.3
- removed net N$9: C4.2, IC1.2, U$3.1
- removed net RD*: IC1.28, U$1.82
- removed net SIWUA: IC1.30
- removed net USB_UART_RX: IC1.39, U$1.12
- removed net USB_UART_TX: IC1.38, U$1.11
- removed net VCC1V8_D: C20.A, IC1.12, IC1.37, IC1.49, IC1.64
- removed net WR*: IC1.29, U$1.81
- new net ESP_UART_RX: U$1.12, U$3.4
- new net ESP_UART_TX: U$1.11, U$3.3
- new net FLASHING: U$3.14
- net GND: now also U$3.1, U$3.12; no longer C20.C, C21.C, C22.C, C23.2, C24.2, C25.1, C26.1, C27.1, C28.1, C4.1, C5.2, C6.1, IC1.1, IC1.10, IC1.11, IC1.13, IC1.15, IC1.25, IC1.35, IC1.47, IC1.5, IC1.51, IC2.5, R9.2, U$3.2, U$3.4, USB1.P5
- net VDD3V3_D: now also C3.1, U$3.6, U$3.8; no longer C25.2, C26.2, C27.2, C28.2, C5.1, IC1.20, IC1.31, IC1.42, IC1.50, IC1.56, IC2.8, L1.2, L2.2, LED2.A, LED3.A, R4.2, R5.2, R6.2, R8.2
- net VDD5V0_D: no longer C6.2, USB1.P1
Routing:
- net VCC1V8_D: track 31.0 -> 0.00 mm
- net N$12: track 28.4 -> 0.00 mm, vias 2 -> 0
- net USB_UART_RX: track 28.3 -> 0.00 mm, vias 2 -> 0
- net USB_UART_TX: track 26.4 -> 0.00 mm, vias 2 -> 0
- net D3: track 25.3 -> 0.00 mm, vias 2 -> 0
- net A0: track 24.9 -> 0.00 mm, vias 2 -> 0
- net N$13: track 23.5 -> 0.00 mm, vias 2 -> 0
- net D4: track 23.2 -> 0.00 mm, vias 2 -> 0
- net ESP_UART_RX: track 0.00 -> 22.7 mm, vias 0 -> 2
- net D7: track 22.5 -> 0.00 mm, vias 2 -> 0
- net VDD3V3_D: track 64.5 -> 85.9 mm, vias 21 -> 10
- net D6: track 20.4 -> 0.00 mm, vias 2 -> 0
- net ESP_UART_TX: track 0.00 -> 20.3 mm, vias 0 -> 2
- net D5: track 18.9 -> 0.00 mm, vias 2 -> 0
- net N$18: track 18.4 -> 0.00 mm, vias 2 -> 0
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Other:
- board text added: "SEAD Light Unit v1 (c) Pavlo Manovi - 2015 sead.systems / pavlo.me"
- board text removed: "SEAD DAQ Unit v2.0b (c) Pavlo Manovi - 2014 sead.systems / pavlo.me"
